File: motor Controller4.brd (EAGLE design)
At the start: 153.7 x 59.4 mm, 50 parts, among them IC1 MEGA8-P, J1 NMJ6HCD2-RM, Q1 IRF540

Commit message: Ver.5 Prep for second print
Routing:
- net GND: track 6.66 -> 11.0 mm
Changed lines of the file:
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@@
 <wire x1="46.99" y1="39.37" x2="50.8" y2="43.18" width="2.54" layer="16"/>
 <wire x1="50.8" y1="43.18" x2="50.8" y2="44.45" width="2.54" layer="16"/>
+<wire x1="43.56" y1="53.34" x2="45.9290875" y2="50.9709125" width="0.1524" layer="1"/>
+<wire x1="45.9290875" y1="50.9709125" x2="45.9290875" y2="49.95080625" width="0.1524" layer="1"/>
+<wire x1="50.8" y1="44.45" x2="45.9290875" y2="49.95080625" width="0" layer="19" extent="1-1"/>
 </signal>
 <signal name="XTAL2">
@@
 <contactref element="U$1" pad="P$2"/>
 <wire x1="6.35" y1="15.24" x2="26.67" y2="15.24" width="0.8128" layer="1"/>
-<wire x1="26.67" y1="15.24" x2="29.21" y2="12.7" width="0.8128" layer="1"/>
-<wire x1="26.67" y1="15.24" x2="34.29" y2="22.86" width="0.8128" layer="1"/>
-<wire x1="34.29" y1="22.86" x2="34.29" y2="39.37" width="0.8128" layer="1"/>
+<wire x1="26.67" y1="15.24" x2="26.72449375" y2="15.18550625" width="0.8128" layer="1"/>
+<wire x1="26.72449375" y1="15.18550625" x2="29.21" y2="12.7" width="0.8128" layer="1"/>
+<wire x1="26.72449375" y1="15.18550625" x2="34.29" y2="22.7510125" width="0.8128" layer="1"/>
+<wire x1="34.29" y1="22.7510125" x2="34.29" y2="39.37" width="0.8128" layer="1"/>
 <wire x1="27.56" y1="45.973" x2="31.75" y2="41.783" width="0.8128" layer="16"/>
 <wire x1="27.56" y1="45.973" x2="27.56" y2="53.34" width="0.8128" layer="16"/>
