File: motor Controller4.sch (EAGLE design)
At the start: 50 parts, among them IC1 MEGA8-P, J1 NMJ6HCD2-RM, Q1 IRF540

Commit message: Ver.5 Prep for second print
Other:
- moved on the sheet: CAL._HEADER
