File: Motor Controller V.5.2.brd (EAGLE design)
At the start: 139 x 58 mm, 52 parts, among them IC1 MEGA8-P, J1 NMJ6HCD2-RM, Q1 IRF540

Commit message: Add ver 5.2 board design
Parts:
- removed 1N5408: 1N5408, diode:DO201-15
- removed LED2: (no value), led:LED3MM
- removed OK1: SFH618A-3, optocoupler:DIP4
- removed VOLTAGE_REGULATOR1: 7805TV, linear:TO220V
- added 5V_POWER_IND: (no value), led:LED3MM
- added D3: 1N5408, diode:DO201-15
- added IC2: SFH618A-3, optocoupler:DIP4
- added LM7805: 7805TV, linear:TO220V
- R4: device rcl:VTA52 -> Benson Motor Controller:VTA52
- moved C1 50.8 mm to (11.6, 8.59), turned to 90 degrees
- moved U$2 45.3 mm to (66.6, 19.6)
- moved Q1 41.0 mm to (129.8, 24.9)
- moved C3 22.5 mm to (84.2, 6.06)
- moved L2 21.1 mm to (26.7, 10.9), turned to 109.5 degrees
- moved C2 18.4 mm to (92.1, 18.8)
- moved CY1 14.2 mm to (47.3, 16.7), turned to 270 degrees
- moved C7 13.3 mm to (42.5, 42.7)
- moved R8 11.2 mm to (94.5, 10.8), turned to 227.3 degrees
- moved C6 10.9 mm to (85.0, 32.6), turned to 0 degrees
- moved F1 9.89 mm to (110.3, 19.6)
- moved MOTOR_CONNECTOR 6.31 mm to (106.9, 3.10)
- moved C15 6.19 mm to (77.5, 32.7), turned to 0 degrees
- moved PS1 5.92 mm to (56.3, 7.23)
- moved LED1 5.30 mm to (74.8, 2.36)
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- renumbered U$3 to PWM_IND
Connections:
- removed net 24VINDGND: IC1.11
- removed net N$18: OK1.4, VOLTAGE_REGULATOR1.3
- net +24V: now also LM7805.1; no longer VOLTAGE_REGULATOR1.1
- net 5VHIGHSIDE: now also IC2.4, LM7805.3
- net 5VINDGND: now also 5V_POWER_IND.A; no longer LED2.A
- net GND: now also IC2.2; no longer OK1.2
- net GNDA: now also LM7805.2; no longer VOLTAGE_REGULATOR1.2
- net MOTOR+: now also D3.C; no longer 1N5408.C
- net MOTOR-: now also D3.A; no longer 1N5408.A
- net N$1: now also IC2.1; no longer OK1.1
- net N$12: now also 5V_POWER_IND.K; no longer LED2.K
- net N$2: now also IC2.3; no longer OK1.3
- net SHIELDINT: now also IC1.12; no longer IC1.14
- net TIPINT: now also IC1.14; no longer IC1.12
Routing:
- net +5V: track 11.2 -> 112.5 mm
- net AC(N): track 0.00 -> 86.1 mm
- net CALIBRATIONPIN: track 0.00 -> 74.2 mm, vias 0 -> 2
- net N$4: track 0.00 -> 65.0 mm
- net RESET: track 0.00 -> 61.3 mm, vias 0 -> 1
- net POWERPIN: track 7.96 -> 66.4 mm
- net +24V: track 0.00 -> 55.7 mm
- net N$9: track 0.00 -> 54.2 mm
- net TIPINT: track 0.00 -> 49.8 mm
- net SHIELDINT: track 0.00 -> 49.7 mm, vias 0 -> 2
- net SPEEDPIN: track 9.96 -> 59.0 mm, vias 0 -> 1
- net N$10: track 0.00 -> 48.3 mm
- net N$6: track 0.00 -> 44.9 mm
- net RINGINT: track 0.00 -> 44.9 mm, vias 0 -> 2
- net MOTOR-: track 0.00 -> 42.0 mm
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Other:
- board text added: "1A/300V"
- board text added: "630mA/250V"
- board text added: "IRF 540"
- board text added: "LM7805"
- board text added: "M+"
- board text added: "M-"
- board text added: "V5.2 DC Motor Controller"
- board text removed: "V.1 DC Motor Control"
