File: Motor Controller V.5.2.sch (EAGLE design)
At the start: 52 parts, among them IC1 MEGA8-P, J1 NMJ6HCD2-RM, Q1 IRF540

Commit message: Add ver 5.2 board design
Parts:
- R4: device rcl:R-US_VTA52 -> Benson Motor Controller:BIGRESISTOR
- renumbered 1N5408 to D3, LED2 to 5V_POWER_IND, OK1 to IC2, U$3 to PWM_IND, VOLTAGE_REGULATOR1 to LM7805
Connections:
- removed net 24VINDGND: IC1.PD5(T1)
- net SHIELDINT: now also IC1.PD6(AIN0); no longer IC1.PB0(ICP)
- net TIPINT: now also IC1.PB0(ICP); no longer IC1.PD6(AIN0)
